Commit message: Pass the new interface parameters through the xacro macros
command_fallback and optional had to be written as raw param tags. Both are
omitted when left empty, so existing descriptions produce identical output.

File: beckhoff_ads_bringup/urdf/beckhoff_bot/beckhoff_ads_interfaces.ros2_control.xacro (robot description, xacro)
@@ -1,5 +1,5 @@
 <?xml version="1.0" encoding="UTF-8"?>
 <robot xmlns:xacro="http://wiki.ros.org/xacro">
-    <xacro:macro name="command_interface_PLC" params="name initial_value:='' PLC_symbol PLC_type n_elements:=1 index:=''">
+    <xacro:macro name="command_interface_PLC" params="name initial_value:='' PLC_symbol PLC_type n_elements:=1 index:='' command_fallback:='' optional:=''">
         <command_interface name="${name}">
             <xacro:if value="${initial_value != ''}">
@@ -12,7 +12,13 @@
                 <param name="index">${index}</param>
             </xacro:if>
+            <xacro:if value="${command_fallback != ''}">
+                <param name="command_fallback">${command_fallback}</param>
+            </xacro:if>
+            <xacro:if value="${optional != ''}">
+                <param name="optional">${optional}</param>
+            </xacro:if>
         </command_interface>
     </xacro:macro>
-    <xacro:macro name="state_interface_PLC" params="name PLC_symbol PLC_type n_elements:=1 index:=''">
+    <xacro:macro name="state_interface_PLC" params="name PLC_symbol PLC_type n_elements:=1 index:='' optional:=''">
         <state_interface name="${name}">
             <param name="PLC_symbol">${PLC_symbol}</param>
@@ -22,4 +28,7 @@
                 <param name="index">${index}</param>
             </xacro:if>
+            <xacro:if value="${optional != ''}">
+                <param name="optional">${optional}</param>
+            </xacro:if>
         </state_interface>
     </xacro:macro>

Commit message: Hard-fault when a critical state item fails past the grace window
A single failing item held its state interface at the last value
forever while read() kept returning healthy; only all items failing
tripped the outage path. Right for telemetry, wrong for a joint
position feeding a closed loop. Joint position and velocity interfaces
now default to critical: a critical item failing beyond the grace
window hard-faults the component. The critical interface parameter
overrides the default in either direction and the xacro state macro
passes it through.

File: beckhoff_ads_bringup/urdf/beckhoff_bot/beckhoff_ads_interfaces.ros2_control.xacro (robot description, xacro)
@@ -20,5 +20,5 @@
         </command_interface>
     </xacro:macro>
-    <xacro:macro name="state_interface_PLC" params="name PLC_symbol PLC_type n_elements:=1 index:='' optional:=''">
+    <xacro:macro name="state_interface_PLC" params="name PLC_symbol PLC_type n_elements:=1 index:='' optional:='' critical:=''">
         <state_interface name="${name}">
             <param name="PLC_symbol">${PLC_symbol}</param>
@@ -31,4 +31,7 @@
                 <param name="optional">${optional}</param>
             </xacro:if>
+            <xacro:if value="${critical != ''}">
+                <param name="critical">${critical}</param>
+            </xacro:if>
         </state_interface>
     </xacro:macro>
